Commit message: omni.urdf

File: touch_description/urdf/omni.urdf (robot description, URDF)
Before this commit: robot phantom_touch, 7 links, 6 joints
Links:
- link base: geometry visual mesh filename=package://omni_description/meshes/base.stl
- link lower_arm: geometry visual mesh filename=package://omni_description/meshes/lower_arm.stl
- link stylus: geometry visual mesh filename=package://omni_description/meshes/pen.stl
- link tip: geometry visual mesh filename=package://omni_description/meshes/tip.stl
- link torso: geometry visual mesh filename=package://omni_description/meshes/torso.stl
- link upper_arm: geometry visual mesh filename=package://omni_description/meshes/upper_arm.stl
- link wrist: geometry visual mesh filename=package://omni_description/meshes/wrist.stl

Commit message: add omni.urdf

File: touch_description/urdf/omni.urdf (robot description, URDF)
Before this commit: robot phantom_omni, 7 links, 6 joints
Links:
- link base: geometry visual mesh filename=package://touch_description/meshes/base.stl
- link lower_arm: geometry visual mesh filename=package://touch_description/meshes/lower_arm.stl
- link stylus: geometry visual mesh filename=package://touch_description/meshes/pen.stl
- link tip: geometry visual mesh filename=package://touch_description/meshes/tip.stl
- link torso: geometry visual mesh filename=package://touch_description/meshes/torso.stl
- link upper_arm: geometry visual mesh filename=package://touch_description/meshes/upper_arm.stl
- link wrist: geometry visual mesh filename=package://touch_description/meshes/wrist.stl
