Commit message: update Touch's URDF

File: touch_description/urdf/touch.urdf (robot description, URDF)
Before this commit: robot phantom_touch, 7 links, 6 joints
Links:
- added link base_ref
- added link stylus_ref
Joints:
- added joint base_fixed: type fixed, parent base, child base_ref, origin xyz=0 0.156 0.090 rpy=1.5708 0 3.1416
- added joint stylus_fixed: type fixed, parent stylus, child stylus_ref, origin xyz=0 0 0 rpy=1.5708 0 0
- joint elbow: limit lower=-0.81 upper=1.25 effort=5 velocity=100 -> lower=-0.81 upper=1.2 effort=5 velocity=100
- joint pitch: limit lower=-0.5 upper=1.75 effort=5 velocity=100 -> lower=0 upper=2.40 effort=5 velocity=100; origin xyz=0 0.0525 0 rpy=0.5 0 0 -> xyz=0 0.0525 0 rpy=0 0 0
- joint yaw: limit lower=3.92 upper=8.83 effort=5 velocity=100 -> lower=-2.50 upper=2.50 effort=5 velocity=100

Commit message: update Touch URDF

File: touch_description/urdf/touch.urdf (robot description, URDF)
Before this commit: robot phantom_touch, 9 links, 8 joints
Joints:
- joint base_fixed: origin xyz=0 0.156 0.090 rpy=1.5708 0 3.1416 -> xyz=0 0.155 0.090 rpy=1.5708 0 3.1416

Commit message: update URDF

File: touch_description/urdf/touch.urdf (robot description, URDF)
Before this commit: robot phantom_touch, 9 links, 8 joints
Joints:
- joint base_fixed: origin xyz=0 0.155 0.090 rpy=1.5708 0 3.1416 -> xyz=0 0.157 0.090 rpy=1.5708 0 3.1416

Commit message: update 22/11/3

File: touch_description/urdf/touch.urdf (robot description, URDF)
Before this commit: robot phantom_touch, 9 links, 8 joints
Links:
- added link probe
Joints:
- added joint probe_fixed: type fixed, parent stylus_ref, child probe, origin xyz=0 0 0 rpy=3.14159 0 0

Commit message: update hardware_interface

File: touch_description/urdf/touch.urdf (robot description, URDF)
Before this commit: robot phantom_touch, 10 links, 9 joints
Joints:
- removed joint elbow
- removed joint pitch
- removed joint roll
- removed joint shoulder
- removed joint waist
- removed joint yaw
- added joint joint1_waist: type revolute, parent base, child torso, origin xyz=0 0 0.09 rpy=0 0 0, axis 0 0 1, limit lower=-0.98 upper=0.98 effort=5 velocity=100
- added joint joint2_shoulder: type revolute, parent torso, child upper_arm, origin xyz=-0.0075 0 0.035 rpy=0 0 0, axis 1 0 0, limit lower=0 upper=1.75 effort=5 velocity=100
- added joint joint3_elbow: type revolute, parent upper_arm, child lower_arm, origin xyz=0.0075 .134 0 rpy=-1.5 0 0, axis 1 0 0, limit lower=-0.81 upper=1.2 effort=5 velocity=100
- added joint joint4_yaw: type revolute, parent lower_arm, child wrist, origin xyz=0 0.08 0, axis 0 1 0, limit lower=-2.50 upper=2.50 effort=5 velocity=100
- added joint joint5_pitch: type revolute, parent wrist, child tip, origin xyz=0 0.0525 0 rpy=0 0 0, axis 1 0 0, limit lower=0 upper=2.40 effort=5 velocity=100
- added joint joint6_roll: type revolute, parent tip, child stylus, origin xyz=0 -0.023 0 rpy=3.14159 3.14159 0, axis 0 1 0, limit lower=-2.58 upper=2.58 effort=5 velocity=100

Commit message: try to apply to Touch effort controller

File: touch_description/urdf/touch.urdf (robot description, URDF)
Before this commit: robot phantom_touch, 10 links, 9 joints
Links:
- added link end_effector
Joints:
- added joint eef_fixed: type fixed, parent lower_arm, child end_effector, origin xyz=0 0.1325 0.0 rpy=0 0 0
